File: Revue Sprint 3/LumCo Carte élec/Carte élec Lum/Carte élec Lum.kicad_pcb (KiCad board)
At the start: 2 copper layers, 59 x 40 mm, 5 parts, among them J1 Autocom4, J2 Autocom2, J3 Autocom2, U1 ESP32-WROOM-32

Commit message: 1
Routing:
- net DI: vias 0 -> 2
- net (no net): vias 0 -> 2
Other:
- board size 59 x 40 mm -> 59 x 48.8 mm
Changed lines of the file:
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@@
 		)
 		(fp_text user "Ext."
-			(at 3.3 1 360)
+			(at 3.3 1 0)
 			(layer "F.Fab")
 			(effects
@@
 		)
 		(fp_text user "${REFERENCE}"
-			(at 0 1.27 360)
+			(at 0 1.27 0)
 			(layer "F.Fab")
 			(effects
@@
 		)
 		(fp_text user "Ext."
-			(at 3.3 3.7 360)
+			(at 3.3 3.7 0)
 			(layer "F.Fab")
 			(effects
@@
 		)
 		(fp_text user "${REFERENCE}"
-			(at 0 3.81 360)
+			(at 0 3.81 0)
 			(layer "F.Fab")
 			(effects
@@
 		(tags "HE14 header THT 1x02 2.54mm single row")
 		(property "Reference" "J3"
-			(at 0.5 -2.5 360)
+			(at 0.5 -2.5 0)
 			(layer "F.SilkS")
 			(effects
@@
 		)
 		(property "Value" "Autocom2"
-			(at 0.3 5.1 360)
+			(at 0.3 5.1 0)
 			(layer "F.Fab")
 			(effects
@@
 		)
 		(property "Footprint" "FootprintGamelGe2_v8.0:Autocom2"
-			(at 0 0 360)
+			(at 0 0 0)
 			(layer "F.Fab")
 			(hide yes)
@@
 		)
 		(property "Datasheet" ""
-			(at 0 0 360)
+			(at 0 0 0)
 			(layer "F.Fab")
 			(hide yes)
@@
 		)
 		(property "Description" "Autocom HE14 connector, single row, 01x02"
-			(at 0 0 360)
+			(at 0 0 0)
 			(layer "F.Fab")
 			(hide yes)
@@
 	)
 	(gr_line
-		(start 141 74)
-		(end 200 74)
+		(start 141 69.2)
+		(end 200 69.2)
 		(stroke
 			(width 0.05)
@@
 	)
 	(gr_line
-		(start 141 114)
-		(end 141 74)
+		(start 141 118)
+		(end 141 69.2)
 		(stroke
 			(width 0.05)
@@
 	)
 	(gr_line
-		(start 200 74)
-		(end 200 114)
+		(start 200 69.2)
+		(end 200 118)
 		(stroke
 			(width 0.05)
@@
 	)
 	(gr_line
-		(start 200 114)
-		(end 141 114)
+		(start 200 118)
+		(end 141 118)
 		(stroke
 			(width 0.05)
@@
 		(layer "Edge.Cuts")
 	)
+	(via
+		(at 197.25 71.95)
+		(size 4.5)
+		(drill 3)
+		(layers "F.Cu" "B.Cu")
+		(net 0)
+	)
+	(via
+		(at 143.75 115.25)
+		(size 4.5)
+		(drill 3)
+		(layers "F.Cu" "B.Cu")
+		(net 0)
+	)
 	(segment
 		(start 149 111)
@@
 		(width 0.9)
 		(layer "F.Cu")
+		(net 5)
+	)
+	(via
+		(at 197.25 115.25)
+		(size 4.5)
+		(drill 3)
+		(layers "F.Cu" "B.Cu")
+		(net 5)
+	)
+	(via
+		(at 143.75 71.95)
+		(size 4.5)
+		(drill 3)
+		(layers "F.Cu" "B.Cu")
 		(net 5)
 	)
@@
 		(polygon
 			(pts
-				(xy 141 74) (xy 200 74) (xy 200 114) (xy 141 114)
-			)
-		)
+				(xy 141 69.2) (xy 200 69.2) (xy 200 118) (xy 141 118)
+			)
+		)
