File: Revue Sprint 3/LumCo Carte élec/Carte élec Lum/Carte élec Lum.kicad_pcb (KiCad board)
At the start: 2 copper layers, 59 x 48.8 mm, 5 parts, among them J1 Autocom4, J2 Autocom2, J3 Autocom2, U1 ESP32-WROOM-32

Commit message: 2
Connections:
- U1 pad 18: CI -> unconnected-(U1-CMD_DNC-Pad18)
- U1 pad 23: DI -> unconnected-(U1-GPIO15-Pad23)
- U1 pad 30: unconnected-(U1-GPIO18-Pad30) -> CI
- U1 pad 37: unconnected-(U1-GPIO23-Pad37) -> DI
Routing:
- net CI: track 8.59 -> 85.8 mm
- net DI: track 49.8 -> 77.0 mm
Changed lines of the file:
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@@
 	(net 6 "unconnected-(U1-GPIO21-Pad33)")
 	(net 7 "unconnected-(U1-GPIO35-Pad6)")
-	(net 8 "unconnected-(U1-GPIO23-Pad37)")
+	(net 8 "unconnected-(U1-CMD_DNC-Pad18)")
 	(net 9 "unconnected-(U1-GPIO25-Pad9)")
 	(net 10 "unconnected-(U1-GPIO03-Pad34)")
@@
 	(net 36 "unconnected-(U1-GPIO12-Pad13)")
 	(net 37 "unconnected-(U1-CLK_DNC-Pad20)")
-	(net 38 "unconnected-(U1-GPIO18-Pad30)")
+	(net 38 "unconnected-(U1-GPIO15-Pad23)")
 	(net 39 "unconnected-(U1-3.3V-Pad1)")
 	(footprint "FootprintGamelGe2_v8.0:Autocom2"
@@
 			(layers "*.Cu" "*.Mask")
 			(remove_unused_layers no)
-			(net 4 "CI")
+			(net 8 "unconnected-(U1-CMD_DNC-Pad18)")
 			(pinfunction "CMD_DNC")
 			(pintype "bidirectional")
@@
 			(layers "*.Cu" "*.Mask")
 			(remove_unused_layers no)
-			(net 5 "DI")
+			(net 38 "unconnected-(U1-GPIO15-Pad23)")
 			(pinfunction "GPIO15")
 			(pintype "bidirectional")
@@
 			(layers "*.Cu" "*.Mask")
 			(remove_unused_layers no)
-			(net 38 "unconnected-(U1-GPIO18-Pad30)")
+			(net 4 "CI")
 			(pinfunction "GPIO18")
 			(pintype "bidirectional")
@@
 			(layers "*.Cu" "*.Mask")
 			(remove_unused_layers no)
-			(net 8 "unconnected-(U1-GPIO23-Pad37)")
+			(net 5 "DI")
 			(pinfunction "GPIO23")
 			(pintype "bidirectional")
@@
 	)
 	(segment
-		(start 192.04 107.9)
-		(end 193.46 106.48)
+		(start 192.04 106.39)
+		(end 190.4 104.75)
 		(width 0.9)
 		(layer "B.Cu")
@@
 	)
 	(segment
+		(start 190.4 104.75)
+		(end 185.929898 104.75)
+		(width 0.9)
+		(layer "B.Cu")
+		(net 4)
+	)
+	(segment
+		(start 147.85 100.23)
+		(end 148.53 99.55)
+		(width 0.9)
+		(layer "B.Cu")
+		(net 4)
+	)
+	(segment
 		(start 192.04 109.5)
-		(end 192.04 107.9)
+		(end 192.04 106.39)
 		(width 0.9)
 		(layer "B.Cu")
@@
 	)
 	(segment
-		(start 193.46 106.48)
-		(end 193.46 101.5)
+		(start 148.83 103.75)
+		(end 147.85 102.77)
+		(width 0.9)
+		(layer "B.Cu")
+		(net 4)
+	)
+	(segment
+		(start 150.05 99.55)
+		(end 170.6 79)
+		(width 0.9)
+		(layer "B.Cu")
+		(net 4)
+	)
+	(segment
+		(start 170.6 79)
+		(end 170.6 76.1)
+		(width 0.9)
+		(layer "B.Cu")
+		(net 4)
+	)
+	(segment
+		(start 148.53 99.55)
+		(end 150.05 99.55)
+		(width 0.9)
+		(layer "B.Cu")
+		(net 4)
+	)
+	(segment
+		(start 184.929898 103.75)
+		(end 148.83 103.75)
+		(width 0.9)
+		(layer "B.Cu")
+		(net 4)
+	)
+	(segment
+		(start 147.85 102.77)
+		(end 147.85 100.23)
+		(width 0.9)
+		(layer "B.Cu")
+		(net 4)
+	)
+	(segment
+		(start 185.929898 104.75)
+		(end 184.929898 103.75)
 		(width 0.9)
 		(layer "B.Cu")
@@
 	)
 	(segment
-		(start 189.5 111.5)
-		(end 190 112)
+		(start 189 106.35)
+		(end 185.55 106.35)
 		(width 0.9)
 		(layer "B.Cu")
@@
 	)
 	(segment
-		(start 188.38 78.88)
-		(end 188.38 76.1)
+		(start 152.82 78.88)
+		(end 152.82 76.1)
 		(width 0.9)
 		(layer "B.Cu")
@@
 	)
 	(segment
-		(start 198.5 109.5)
-		(end 198.5 89)
+		(start 146.45 85.25)
+		(end 152.82 78.88)
 		(width 0.9)
 		(layer "B.Cu")
@@
 	)
 	(segment
-		(start 198.5 89)
-		(end 188.38 78.88)
+		(start 189.5 106.85)
+		(end 189 106.35)
 		(width 0.9)
 		(layer "B.Cu")
@@
 	)
 	(segment
-		(start 190 112)
-		(end 196 112)
+		(start 148.250101 105.15)
+		(end 146.45 103.349899)
 		(width 0.9)
 		(layer "B.Cu")
@@
 	)
 	(segment
+		(start 184.35 105.15)
+		(end 148.250101 105.15)
+		(width 0.9)
+		(layer "B.Cu")
+		(net 5)
+	)
+	(segment
+		(start 146.45 103.349899)
+		(end 146.45 85.25)
+		(width 0.9)
+		(layer "B.Cu")
+		(net 5)
+	)
+	(segment
 		(start 189.5 109.5)
-		(end 189.5 111.5)
+		(end 189.5 106.85)
 		(width 0.9)
 		(layer "B.Cu")
@@
 	)
 	(segment
-		(start 196 112)
-		(end 198.5 109.5)
+		(start 185.55 106.35)
+		(end 184.35 105.15)
 		(width 0.9)
 		(layer "B.Cu")
@@
 		(filled_areas_thickness no)
 		(fill yes
-			(thermal_gap 0.508)
-			(thermal_bridge_width 0.508)
-			(island_removal_mode 1)
-			(island_area_min 10)
+			(thermal_gap 0.5)
+			(thermal_bridge_width 0.5)
 		)
 		(polygon
