File: Revue Sprint 3/LumCo Carte élec/Carte élec Lum/Carte élec Lum.kicad_sch (KiCad schematic)
At the start: 5 parts, among them J1 Autocom4, J2 Autocom2, J3 Autocom2, U1 ESP32-WROOM-32

Commit message: fond
Connections:
- net 5Vss renamed 5V
Changed lines of the file:
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@@
 		)
 	)
-	(global_label "5Vss"
+	(global_label "5V"
 		(shape input)
 		(at 34.29 20.32 0)
@@
 		)
 		(property "Intersheetrefs" "${INTERSHEET_REFS}"
-			(at 41.6295 20.32 0)
+			(at 39.5733 20.32 0)
 			(effects
 				(font
@@
 		)
 	)
-	(global_label "5Vss"
+	(global_label "5V"
 		(shape input)
 		(at 35.56 52.07 180)
@@
 		)
 		(property "Intersheetrefs" "${INTERSHEET_REFS}"
-			(at 28.2205 52.07 0)
+			(at 30.2767 52.07 0)
 			(effects
 				(font

Commit message: 2
Connections:
- net CI: now also U1.30 (GPIO18); no longer U1.18 (CMD_DNC)
- net DI: now also U1.37 (GPIO23); no longer U1.23 (GPIO15)
Changed lines of the file:
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@@
 	(global_label "CI"
 		(shape input)
-		(at 35.56 76.2 180)
-		(fields_autoplaced yes)
-		(effects
-			(font
-				(size 1.27 1.27)
-			)
-			(justify right)
-		)
-		(property "Intersheetrefs" "${INTERSHEET_REFS}"
-			(at 30.7 76.2 0)
-			(effects
-				(font
-					(size 1.27 1.27)
-				)
-				(justify right)
+		(at 66.04 83.82 0)
+		(fields_autoplaced yes)
+		(effects
+			(font
+				(size 1.27 1.27)
+			)
+			(justify left)
+		)
+		(property "Intersheetrefs" "${INTERSHEET_REFS}"
+			(at 70.9 83.82 0)
+			(effects
+				(font
+					(size 1.27 1.27)
+				)
+				(justify left)
 				(hide yes)
 			)
@@
 	(global_label "DI"
 		(shape input)
-		(at 66.04 66.04 0)
-		(fields_autoplaced yes)
-		(effects
-			(font
-				(size 1.27 1.27)
-			)
-			(justify left)
-		)
-		(property "Intersheetrefs" "${INTERSHEET_REFS}"
-			(at 70.9 66.04 0)
-			(effects
-				(font
+		(at 66.04 99.06 0)
+		(fields_autoplaced yes)
+		(effects
+			(font
+				(size 1.27 1.27)
+			)
+			(justify left)
+		)
+		(property "Intersheetrefs" "${INTERSHEET_REFS}"
+			(at 70.9 99.06 0)
+			(effects
+				(font
